File: lo2.kicad_sch (KiCad schematic)
At the start: 0 parts

Commit message: added labels to LO, duplicated to LO2
Parts:
- added C1, C10, C11, C15, C2, C6: 100nF, ar_passives:C_0402, symbol #bt-db:capacitor/CAPC-00573
- added C12, C13, C14, C7: 1uF, ar_passives:C_0402, symbol #bt-db:capacitor/CAPC-00622
- added C16, C17, C18, C19: 22pF, ar_passives:C_0201, symbol #bt-db:capacitor/CAPC-00021
- added C3, C4, C8: 10uF, ar_passives:C_0402, symbol #bt-db:capacitor/CAPC-00667
- added C5: 470nF, ar_passives:C_0402, symbol #bt-db:capacitor/CAPC-00613
- added C9: 10nF, ar_passives:C_0402, symbol #bt-db:capacitor/CAPC-00514
- added CLF1: 0pF, ar_passives:C_0603, symbol #bt-db:capacitor/CAPC-00674
- added CLF2, CLF3: 0pF, ar_passives:C_0402, symbol #bt-db:capacitor/CAPC-00415
- added RLF2, RLF3: TBD, ar_passives:R_0402, symbol #bt-db:resistor/RESI-00693
- added U3: (no value), ar_ic:QFN40, symbol #bt-db:ic/ICIR-00204
Connections:
- new net: CLF2.1, RLF2.2
- new net CPOut: CLF1.1, RLF2.1, RLF3.2, U3.12 (CPout)
- new net GND: C10.2, C11.2, C12.2, C13.2, C14.2, C15.2, C3.2, C4.2, C5.1, C6.2, C7.2, C8.2, C9.2, CLF1.2, CLF2.2, CLF3.1, U3.13 (GND), U3.14 (GND), U3.2 (GND), U3.25 (GND), U3.31 (GND), U3.34 (GND), U3.39 (GND), U3.4 (GND), U3.40 (GND), U3.6 (GND), U3.EP (GND)
- new net LO1_3V3_BUF: C15.1, U3.21 (VccBUF)
- new net LO1_3V3_SYN: C10.1, C11.1, C12.1, C13.1, C14.1, U3.11 (VccCP), U3.15 (VccMASH), U3.26 (VccVCO2), U3.37 (VccVCO), U3.7 (VccDIG)
- new net LO_A.N: C17.2
- new net LO_A.P: C16.2
- new net LO_B.N: C19.2
- new net LO_B.P: C18.2
- new net OSC_N: C2.2, U3.9 (OSCinM)
- new net OSC_P: C1.2, U3.8 (OSCinP)
- new net REF.N: C2.1
- new net REF.P: C1.1
- new net RF_A_N: C17.1, U3.22 (RFoutAM)
- new net RF_A_P: C16.1, U3.23 (RFoutAP)
- new net RF_B_N: C19.1, U3.18 (RFoutBM)
- new net RF_B_P: C18.1, U3.19 (RFoutBP)
- new net SYN.CE: U3.1 (CE)
- new net SYN.MUX: U3.20 (MUXout)
- new net SYN.RC: U3.30 (RampClk)
- new net SYN.RD: U3.32 (RampDir)
- new net SYN.SCK: U3.16 (SCK)
- new net SYN.SDI: U3.17 (SDI)
- new net SYN.~{CS}: U3.24 (~{CS})
- new net VTUNE: CLF3.2, RLF3.1, U3.35 (Vtune)
- new net VbiasVARAC: C4.1, U3.33 (VbiasVARAC)
- new net VbiasVCO: C5.2, U3.3 (VbiasVCO)
- new net VbiasVCO2: C6.1, U3.27 (VbiasVCO2)
- new net VrefVCO: C3.1, U3.36 (VrefVCO)
- new net VrefVCO2: C8.1, U3.29 (VrefVCO2)
- new net VregIN: C7.1, U3.10 (VregIN)
- new net VregVCO: C9.1, U3.38 (VregVCO)
Other:
- note added: "11"
- note added: "15"
- note added: "26"
- note added: "37"
- note added: "7"
